File: ModuleV440/ModuleV440.kicad_pcb (KiCad board)
At the start: 2 copper layers, 30 x 61.3 mm, 45 parts, among them J2 AVR-ISP-6, Q1 AO3400A, U1 EL3H7(B)(TA)-G, Y1 8MHZ Ceramic Resonator

Commit message: revert copyright change
Other:
- board text added: "©2019-2021 Stuart Pittaway"
- board text removed: "©2019-2022 Stuart Pittaway Matthias Urlichs"
Changed lines of the file:
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@@
   (gr_line (start 103.6976 73.2236) (end 122.5776 73.2236) (layer "Edge.Cuts") (width 0.1))
   (gr_arc (start 130.4426 47.9876) (mid 131.50326 48.42694) (end 131.9426 49.4876) (layer "Edge.Cuts") (width 0.15))
-  (gr_text "©2019-2022\nStuart Pittaway\nMatthias Urlichs" (at 109.6176 87.3376) (layer "B.SilkS")
+  (gr_text "©2019-2021\nStuart Pittaway" (at 109.6176 87.3376) (layer "B.SilkS")
     (effects (font (size 1.2 1.2) (thickness 0.3)) (justify mirror))
   )
