File: ModuleV440/ModuleV440.kicad_sch (KiCad schematic)
At the start: 42 parts

Commit message: property sync, no changes
Parts:
- ATTINY841: value (none) -> ATtiny841-SSU
- C1: value (none) -> 100nF; footprint (none) -> Capacitor_SMD:C_0805_2012Metric
- C2: value (none) -> 1uF; footprint (none) -> Capacitor_SMD:C_0805_2012Metric
- C4, C5: value (none) -> 22pF; footprint (none) -> Capacitor_SMD:C_0805_2012Metric
- D1: value (none) -> AZ432ANTR-E1; footprint (none) -> Package_TO_SOT_SMD:SOT-23
- D2: value (none) -> SMBJ5.0A; footprint (none) -> Diode_SMD:D_SMB
- D3: value (none) -> Red; footprint (none) -> LED_SMD:LED_0805_2012Metric
- D4: value (none) -> Blue; footprint (none) -> LED_SMD:LED_0805_2012Metric
- EXTTEMP1: value (none) -> Ext Temp Sensor; footprint (none) -> Connector_JST:JST_PH_S2B-PH-K_1x02_P2.00mm_Horizontal
- F1: value (none) -> mSMD150; footprint (none) -> Fuse:Fuse_1812_4532Metric
- J2: value (none) -> AVR-ISP-6; footprint (none) -> Pin_Headers:Pin_Header_Straight_2x03_Pitch2.54mm
- POWER1: value (none) -> Battery; footprint (none) -> Connector_JST:JST_PH_S2B-PH-K_1x02_P2.00mm_Horizontal
- Q1: value (none) -> AO3400A; footprint (none) -> TO_SOT_Packages_SMD:SOT-23
- R1, R15, R20, R21: value (none) -> 10KOHMS; footprint (none) -> Resistor_SMD:R_0805_2012Metric
- R12, R22, R24, R25, R26, R29, R30, R6, R8: value (none) -> 3.3OHM 3/4W; footprint (none) -> Resistor_SMD:R_2010_5025Metric
- R14: value (none) -> 510OHMS; footprint (none) -> Resistor_SMD:R_0805_2012Metric
- R16, R17, R18: value (none) -> 2.2KOHMS; footprint (none) -> Resistor_SMD:R_0805_2012Metric
- R19, R23: value (none) -> CMFB103F3950FANT; footprint (none) -> Resistor_SMD:R_0805_2012Metric
- R2: value (none) -> 1KOHMS; footprint (none) -> Resistor_SMD:R_0805_2012Metric
- R3: value (none) -> 6.8K; footprint (none) -> Resistor_SMD:R_0805_2012Metric
- R4: value (none) -> 2.7K; footprint (none) -> Resistor_SMD:R_0805_2012Metric
- R5: value (none) -> 220 OHMS; footprint (none) -> Resistor_SMD:R_0805_2012Metric
- REMOTE1: value (none) -> Ext Temp Sensor; footprint (none) -> Connector_PinHeader_2.54mm:PinHeader_1x02_P2.54mm_Vertical
- RX1: value (none) -> RX Connector; footprint (none) -> Connector_JST:JST_PH_S2B-PH-K_1x02_P2.00mm_Horizontal
- TX1: value (none) -> TX Connector; footprint (none) -> Connector_JST:JST_PH_S2B-PH-K_1x02_P2.00mm_Horizontal
- U1: value (none) -> EL3H7(B)(TA)-G; footprint (none) -> Package_SO:SOP-4_4.4x2.6mm_P1.27mm
- Y1: value (none) -> 8MHZ Ceramic Resonator; footprint (none) -> Crystals:Crystal_SMD_5032-2pin_5.0x3.2mm
