File: ControllerCircuit/ControllerCircuit.kicad_sch (KiCad schematic)
At the start: 80 parts

Commit message: property sync, no changes
Parts:
- C1, C2, C5, C6, C8: value (none) -> 100nF; footprint (none) -> Capacitor_SMD:C_0805_2012Metric
- C10, C9: value (none) -> 1uF; footprint (none) -> Capacitor_SMD:C_0805_2012Metric
- C3, C4: value (none) -> 22uF 6.3V; footprint (none) -> Capacitor_Tantalum_SMD:CP_EIA-3216-18_Kemet-A_Pad1.58x1.35mm_HandSolder
- D1: value (none) -> RGB; footprint (none) -> LED_SMD:LED_RGB_5050-6
- D2, D5: value (none) -> LL4148; footprint (none) -> Diode_SMD:D_MiniMELF
- D3, D4, D6: value (none) -> YELLOW LED; footprint (none) -> LED_SMD:LED_0603_1608Metric_Pad1.05x0.95mm_HandSolder
- D7: value (none) -> D_Zener_Small; footprint (none) -> Diode_THT:D_5W_P10.16mm_Horizontal
- D8: value (none) -> NUP2105LT1G; footprint (none) -> Package_TO_SOT_SMD:SOT-23
- F1: value (none) -> Fuse, 1.85A; footprint (none) -> Fuse:Fuse_2920_7451Metric
- J1, J12, J14, J4, J5, J7: value (none) -> ScrewTerminal; footprint (none) -> ControllerCircuit:Terminal-Block_3.81_4P_LCSC_C395880
- J10: value (none) -> Conn_01x02_Female; footprint (none) -> Connector_PinHeader_2.54mm:PinHeader_1x02_P2.54mm_Horizontal
- J11: value (none) -> Conn_01x03_Female; footprint (none) -> Connector_PinHeader_2.54mm:PinHeader_1x03_P2.54mm_Vertical
- J13, JP2, JP3: value (none) -> Conn_01x02_Female; footprint (none) -> Connector_PinHeader_2.54mm:PinHeader_1x02_P2.54mm_Vertical
- J15: value (none) -> Molex 0472192001; footprint (none) -> 0472192001
- J2, J3: value (none) -> ScrewTerminal3Pin; footprint (none) -> ControllerCircuit:Terminal-Block_5.0mm_3P-LCSC_C395850
- J6: value (none) -> AVR-ISP-6; footprint (none) -> Connector_PinHeader_2.54mm:PinHeader_2x03_P2.54mm_Vertical
- J8: value (none) -> 2x3 2.54mm IDC Connectors; footprint (none) -> Connector_PinHeader_2.54mm:PinHeader_2x03_P2.54mm_Vertical
- J9: value (none) -> Conn_01x06_Female; footprint (none) -> Connector_PinHeader_2.54mm:PinHeader_1x06_P2.54mm_Vertical
- JP1, JP4: value (none) -> OptTermination; footprint (none) -> Jumper:SolderJumper-2_P1.3mm_Open_RoundedPad1.0x1.5mm
- JP5: value (none) -> CANBUS Volt Select; footprint (none) -> Jumper:SolderJumper-3_P1.3mm_Bridged12_RoundedPad1.0x1.5mm
- K1, K2: value (none) -> SRD-05VDC-SL-C
- LCD1: value (none) -> LCD; footprint (none) -> ControllerCircuit:TFTSPI_2_8_240x320_TOUCH
- Q1, Q2: value (none) -> AO3400A; footprint (none) -> Package_TO_SOT_SMD:SOT-23
- Q3: value (none) -> AO3401A; footprint (none) -> Package_TO_SOT_SMD:SOT-23
- R1, R8: value (none) -> 100R; footprint (none) -> Resistor_SMD:R_0805_2012Metric
- R10, R14, R18, R25: value (none) -> 220R; footprint (none) -> Resistor_SMD:R_0805_2012Metric
- R11, R15, R19, R20, R23, R24: value (none) -> 10K; footprint (none) -> Resistor_SMD:R_0805_2012Metric
- R12, R13: value (none) -> 560R; footprint (none) -> Resistor_SMD:R_0805_2012Metric
- R16, R2, R5: value (none) -> 2K2; footprint (none) -> Resistor_SMD:R_0805_2012Metric
- R17, R4: value (none) -> 300R; footprint (none) -> Resistor_SMD:R_0805_2012Metric
- R21, R22, R3: value (none) -> 180R; footprint (none) -> Resistor_SMD:R_0805_2012Metric
- R6, R9: value (none) -> 120R; footprint (none) -> Resistor_SMD:R_0805_2012Metric
- RX1: value (none) -> Receive; footprint (none) -> Connector_JST:JST_PH_S2B-PH-K_1x02_P2.00mm_Horizontal
- TX1: value (none) -> Transmit; footprint (none) -> Connector_JST:JST_PH_S2B-PH-K_1x02_P2.00mm_Horizontal
- U1: value (none) -> TJA1057GT/3; footprint (none) -> Package_SO:SOIC-8_3.9x4.9mm_P1.27mm
- U10: value (none) -> ATtiny841-SSU
- U12, U9: value (none) -> AQY212GSZ; footprint (none) -> Package_SO:SO-4_4.4x3.6mm_P2.54mm
- U2: value (none) -> EL3H7(B)(TA)-G; footprint (none) -> Package_SO:SOP-4_4.4x2.6mm_P1.27mm
- U3: value (none) -> TCA6408APWR; footprint (none) -> Package_SO:TSSOP-16_4.4x5mm_P0.65mm
- U4: value (none) -> ESP32-DEVKITC-32D
- U5: value (none) -> SN65HVD75DR; footprint (none) -> Package_SO:SOIC-8_3.9x4.9mm_P1.27mm
- U6: value (none) -> AMS1117-3.3; footprint (none) -> Package_TO_SOT_SMD:SOT-223-3_TabPin2
- U8: value (none) -> TCA9534A; footprint (none) -> Package_SO:TSSOP-16_4.4x5mm_P0.65mm
