File: ModuleV421/ModuleV421.kicad_pcb (KiCad board)
At the start: 2 copper layers, 30 x 50 mm, 54 parts, among them J2 AVR-ISP-6, Q1 AO3400A, U1 EL3H7(B)(TA)-G

Commit message: spurious hole w/ overlapping courtyard
Parts:
- removed the REF** at (130.4, 92.2)
Changed lines of the file:
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@@
     )
-  )
-  (footprint "Mounting_Holes:MountingHole_2.5mm" locked (layer "F.Cu")
-    (at 130.4176 92.2376)
-    (descr "Mounting Hole 2.5mm, no annular")
-    (tags "mounting hole 2.5mm no annular")
-    (attr exclude_from_pos_files exclude_from_bom)
-    (fp_text reference "REF**" (at 7.5 0.5) (layer "F.SilkS") hide
-      (effects (font (size 1 1) (thickness 0.15)))
-    )
-    (fp_text value "JLCAssemblyHole_1_152mm" (at 0 3.5) (layer "F.Fab")
-      (effects (font (size 1 1) (thickness 0.15)))
-    )
-    (fp_text user "${REFERENCE}" (at 0.3 1.9) (layer "F.Fab")
-      (effects (font (size 1 1) (thickness 0.15)))
-    )
-    (fp_circle (center 0 0) (end 1.16 0) (layer "Cmts.User") (width 0.15) (fill none))
-    (fp_circle (center 0 0) (end 1.16 0) (layer "F.CrtYd") (width 0.05) (fill none))
-    (pad "" np_thru_hole circle locked (at 0 0) (size 1.152 1.152) (drill 1.152) (layers *.Cu *.Mask))
   )
   (footprint "LEDs:LED_0805" (layer "F.Cu")
@@
   (zone (net 1) (net_name "GND") (layer "F.Cu") (hatch edge 0.508)
     (connect_pads (clearance 0.508))
-    (min_thickness 0.254)
+    (min_thickness 0.254) (filled_areas_thickness no)
     (fill yes (thermal_gap 0.508) (thermal_bridge_width 0.508))
     (polygon
@@
   (zone (net 1) (net_name "GND") (layer "B.Cu") (hatch edge 0.508)
     (connect_pads (clearance 0.508))
-    (min_thickness 0.254)
+    (min_thickness 0.254) (filled_areas_thickness no)
     (fill yes (thermal_gap 0.508) (thermal_bridge_width 0.508))
     (polygon
